Commit message: Delete VMC.

File: diablo/urdf/diablo.urdf.xacro (robot description, xacro)
@@ -13,5 +13,5 @@
 <!--        <parent link="world"/>-->
 <!--        <child link="diablo_base_link"/>-->
-<!--        <origin xyz="0 0 0.3" rpy="0 0 0"/>-->
+<!--        <origin xyz="0 0 0.2" rpy="0 0 0"/>-->
 <!--    </joint>-->
     <!--    main link-->

File: diablo/urdf/diablo.xacro (robot description, xacro)
@@ -6,5 +6,5 @@
     <xacro:arg name="fixed_wheel" default="false"/>
     <xacro:arg name="use_gazebo" default="true"/>
-    <xacro:arg name="close_chain" default="false"/>
+    <xacro:arg name="close_chain" default="true"/>
     <xacro:arg name="use_simulation" default="false"/>
     <xacro:if value="$(arg load_chassis)">
